File: v1_0/blinker_v1_0/blinker_v1_0.kicad_sch (KiCad schematic)
At the start: 23 parts, among them J3 Barrel_Jack_Switch_Pin3Ring, Q1 2N7002K, SW1 SW_DIP_x02, SW2 SW_DIP_x02, U1 NE555D, U2 LM1117MP-ADJ

Commit message: lyt started
Parts:
- U2: footprint Package_TO_SOT_SMD:SOT-223 -> Package_TO_SOT_SMD:SOT-223-3_TabPin2
- j1, j2: footprint Connector_Pin:Pin_D1.0mm_L10.0mm_LooseFit -> Connector_Pin:Pin_D1.0mm_L10.0mm
Connections:
- net Uin: now reaches C3.1, J3.1, R7.1, U2.3 (VI)
- net Uin: now also j1.1; no longer j1.
- net at J3.2: now also j2.1; no longer j2.
