File: v1_0/blinker_v1_0/blinker_v1_0.kicad_pcb (KiCad board)
At the start: 2 copper layers, 23 parts, among them J3 Barrel_Jack_Switch_Pin3Ring, Q1 2N7002K, SW1 SW_DIP_x02, SW2 SW_DIP_x02, U1 NE555D, U2 LM1117MP-ADJ

Commit message: lyt started
Parts:
- U2: footprint Package_TO_SOT_SMD:SOT-223 -> Package_TO_SOT_SMD:SOT-223-3_TabPin2
- j1, j2: footprint Connector_Pin:Pin_D1.0mm_L10.0mm_LooseFit -> Connector_Pin:Pin_D1.0mm_L10.0mm
- moved C3 35.8 mm to (164.6, 35.0), turned to 90 degrees
- moved j2 35.0 mm to (173.9, 42.1)
- moved C4 31.4 mm to (160.8, 40.0)
- moved j1 30.9 mm to (168.6, 42.4)
- moved R6 17.1 mm to (155.2, 39.2), turned to 90 degrees
- moved R5 14.7 mm to (157.5, 40.0), turned to 180 degrees
- moved U2 11.6 mm to (159.6, 34.7), turned to 90 degrees
- moved J3 9.21 mm to (167.6, 34.6), turned to 90 degrees
Connections:
- C3 pad 1: Net-(U2-VI) -> /Uin
- J3 pad 1: Net-(U2-VI) -> /Uin
- R7 pad 1: Net-(U2-VI) -> /Uin
- U2 pad 3: Net-(U2-VI) -> /Uin
- j1 pad 1: (no net) -> /Uin
- j2 pad 1: (no net) -> Net-(J3-Pad2)

Commit message: lyt cont, outline is developing
Parts:
- moved C1 27.7 mm to (166.2, 45.7), turned to 90 degrees
- moved D1 18.8 mm to (155.8, 50.2), turned to 180 degrees
- moved U1 18.7 mm to (161.7, 44.7)
- moved R7 17.0 mm to (164.8, 39.8), turned to -90 degrees
- moved R3 17.0 mm to (167.8, 43.2), turned to 90 degrees
- moved C2 16.5 mm to (155.8, 52.0), turned to 180 degrees
- moved SW1 16.1 mm to (152.4, 33.5), turned to -90 degrees
- moved R8 15.7 mm to (156.9, 43.6), turned to -90 degrees
- moved SW2 14.2 mm to (152.4, 43.4), turned to -90 degrees
- moved D2 13.9 mm to (168.8, 48.8), turned to 90 degrees
- moved R9 13.0 mm to (155.6, 48.5)
- moved R2 9.79 mm to (160.8, 49.2), turned to -90 degrees
- moved R1 8.48 mm to (155.6, 47.0)
- moved R4 8.06 mm to (155.2, 43.6), turned to -90 degrees
- moved R6 3.88 mm to (154.9, 35.3)
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Other:
- board outline added: 55.2 x 25.7 mm
